File: PCB/6axis_robot.kicad_pcb (KiCad board)
At the start: 4 copper layers, 124.4 x 115.3 mm, 82 parts, among them J10 Conn_01x03_Socket, J11 Conn_01x03_Socket, J12 Conn_01x03_Socket, J17 1729128, J18 Conn_01x04_Socket, J19 Conn_01x04_Socket, J2 Conn_01x03_Socket, J20 Conn_01x03_Socket, J21 Conn_01x02_Socket, J24 Conn_02x08_Counter_Clockwise, J25 Conn_01x04_Socket, J26 Conn_02x08_Counter_Clockwise, J27 Conn_01x04_Socket, J28 Conn_02x08_Counter_Clockwise, J29 Conn_01x04_Socket, J30 Conn_02x08_Counter_Clockwise, J31 Conn_01x04_Socket, J32 Conn_02x08_Counter_Clockwise, J33 Conn_01x04_Socket, J34 Conn_02x08_Counter_Clockwise, J35 Conn_01x04_Socket, J8 Conn_01x03_Socket, J9 Conn_01x03_Socket, Q10 Q_PMOS_GSD, SW2 SW_Push, U10 SN65HVD230, U11 PC817, U8 AMS1117-3.3, U9 STM32F446RETx, Y3 8MHz

Commit message: Add files via upload
Parts:
- added C29: 100nF, Capacitor_SMD:C_0805_2012Metric, F.Cu at (91.5, 108.0)
- added C3: 10uF, Capacitor_THT:CP_Radial_D6.3mm_P2.50mm, F.Cu at (134.5, 80.2)
- added C30: 100nF, Capacitor_SMD:C_0805_2012Metric, F.Cu at (128.9, 127.2)
- added C31: 10nF, Capacitor_SMD:C_0805_2012Metric, F.Cu at (101.5, 116.2)
- added C32: 22uF, Capacitor_SMD:C_0805_2012Metric, F.Cu at (137.2, 98.0)
- added C33: 22uF, Capacitor_SMD:C_0805_2012Metric, F.Cu at (130.8, 105.2)
- added C34: 10nF, Capacitor_SMD:C_0805_2012Metric, F.Cu at (130.5, 115.8)
- added D1: B340, Diode_SMD:D_SMC, F.Cu at (114.0, 105.2)
- added L1: 10uH, Inductor_SMD:L_Sunlord_SWPA6045S, F.Cu at (73.2, 105.8)
- added R22: 10k, Resistor_SMD:R_0805_2012Metric, F.Cu at (104.4, 104.2)
- added R23: 1.96K, Resistor_SMD:R_0805_2012Metric, F.Cu at (104.4, 107.2)
- added R24: 10k, Resistor_SMD:R_0805_2012Metric, F.Cu at (128.0, 109.5)
- added U1: TPS54331D, footprints:SOIC127P599X175-8N, F.Cu at (96.8, 111.0)
- H1, H2, H3, H4: value M3 -> MountingHole
- J22: renamed from CAN BUS J22
Routing:
- net +5V: track 68.9 -> 175.1 mm, vias 0 -> 2
- net Net-(D1-A): track 0.00 -> 61.9 mm, vias 0 -> 2
- net +24V: track 428.5 -> 487.8 mm, vias 7 -> 9
- net Net-(U1-COMP): track 0.00 -> 34.5 mm, vias 0 -> 2
- net Net-(U1-VSENSE): track 0.00 -> 10.2 mm
- net Net-(U1-BOOT): track 0.00 -> 8.51 mm
- net GND: track 248.0 -> 254.8 mm, vias 51 -> 53
- net Net-(C34-Pad1): track 0.00 -> 6.71 mm
- net Net-(U1-SS): track 0.00 -> 4.91 mm
- net +3V3: track 566.0 -> 570.5 mm, vias 14 -> 16
